Commit message: Gazebo is still broken, simplified model imported.

File: src/annin_ar4_description/urdf/ar.urdf.xacro (robot description, xacro)
@@ -1,8 +1,18 @@
 <?xml version="1.0"?>
-<robot xmlns:xacro="http://wiki.ros.org/xacro" name="$(arg ar_model)">
+<robot xmlns:xacro="http://wiki.ros.org/xacro" name="ar4">
   <!-- <xacro:arg name="tf_prefix" default="" />
   <xacro:arg name="include_gripper" default="true"/> -->
   <!-- <xacro:include filename="$(find annin_ar4_description)/urdf/ar_macro.xacro"/> -->
   <xacro:include filename="$(find annin_ar4_description)/urdf/annin_ar4_geometry.urdf"/>
+  <link name="base_link"/>
+  <joint name="base_joint" type="fixed">
+      <parent link="base_link"/>
+      <child link="baseplate"/>
+  </joint>
+  <link name="world"/>
+  <joint name="world_fixed" type="fixed">
+      <parent link="world"/>
+      <child link="base_link"/>
+  </joint>
   <!-- <link name="world" />
   <xacro:ar_robot
