Commit message: Before replacement

File: src/annin_ar4_description/urdf/ar.ros2_control.xacro (robot description, xacro)
@@ -27,5 +27,6 @@
         <param name="tf_prefix">${tf_prefix}</param>
       </hardware>
-      <joint name="${tf_prefix}joint_1">
+<!-- Joint_1 -->
+      <joint name="${tf_prefix}base_to_link1">
         <command_interface name="position">
           <param name="min">${robot_parameters['j1_limit_min']}</param>
@@ -41,5 +42,6 @@
         <param name="position_offset">${joint_offset_parameters['joint_1']}</param>
       </joint>
-      <joint name="${tf_prefix}joint_2">
+<!-- joint_2 -->
+      <joint name="${tf_prefix}link1_to_link2">
         <command_interface name="position">
           <param name="min">${robot_parameters['j2_limit_min']}</param>
@@ -55,5 +57,6 @@
         <param name="position_offset">${joint_offset_parameters['joint_2']}</param>
       </joint>
-      <joint name="${tf_prefix}joint_3">
+<!-- joint_3 -->
+      <joint name="${tf_prefix}link2_to_link3">
         <command_interface name="position">
           <param name="min">${robot_parameters['j3_limit_min']}</param>
@@ -69,5 +72,6 @@
         <param name="position_offset">${joint_offset_parameters['joint_3']}</param>
       </joint>
-      <joint name="${tf_prefix}joint_4">
+<!-- joint_4 -->
+      <joint name="${tf_prefix}link3_to_end_effector_mount">
         <command_interface name="position">
           <param name="min">${robot_parameters['j4_limit_min']}</param>
@@ -83,5 +87,6 @@
         <param name="position_offset">${joint_offset_parameters['joint_4']}</param>
       </joint>
-      <joint name="${tf_prefix}joint_5">
+<!-- joint_5 -->
+      <joint name="${tf_prefix}endeffector_mount">
         <command_interface name="position">
           <param name="min">${robot_parameters['j5_limit_min']}</param>
@@ -97,5 +102,6 @@
         <param name="position_offset">${joint_offset_parameters['joint_5']}</param>
       </joint>
-      <joint name="${tf_prefix}joint_6">
+<!-- joint_6 -->
+      <joint name="${tf_prefix}endeffector">
         <command_interface name="position">
           <param name="min">${robot_parameters['j6_limit_min']}</param>

File: src/annin_ar4_description/urdf/ar.urdf.xacro (robot description, xacro)
@@ -4,5 +4,5 @@
   <xacro:arg name="include_gripper" default="true"/> -->
   <!-- <xacro:arg name="tf_prefix" default="" /> -->
-  <!-- <xacro:include filename="$(find annin_ar4_description)/urdf/ar_macro.xacro"/> -->
+  <xacro:include filename="$(find annin_ar4_description)/urdf/ar.ros2_control.xacro"/>
   <xacro:include filename="$(find annin_ar4_description)/urdf/annin_ar4_geometry.urdf"/>
   <link name="base_link"/>
@@ -31,14 +31,22 @@
     />
   </xacro:if> -->
-  <ros2_control name="GazeboSystem" type="system">
-  <hardware>
-    <plugin>gazebo_ros2_control/GazeboSystem</plugin>
-  </hardware>
-  <joint name="head_swivel" />
-</ros2_control>
-<gazebo>
-  <plugin filename="libgazebo_ros2_control.so" name="gazebo_ros2_control">
-    <parameters>$(find urdf_sim_tutorial)/config/09a-minimal.yaml</parameters>
-  </plugin>
-</gazebo>
+  <!-- <gazebo reference="world" />
+  <gazebo>
+    <plugin filename="libgz_ros2_control-system" name="gz_ros2_control::GazeboSimROS2ControlPlugin">
+      <parameters>$(arg simulation_controllers)</parameters>
+      <ros>
+        <namespace>$(arg namespace)</namespace>
+      </ros>
+    </plugin>
+  </gazebo> -->
+  <xacro:ar_ros2_control
+    ar_model="$(arg ar_model)"
+    plugin_name="gz_ros2_control/GazeboSimSystem"
+    serial_port="None"
+    calibrate="False"
+    robot_parameters_file="$(find annin_ar4_description)/config/$(arg ar_model).yaml"
+    joint_offset_parameters_file="$(find annin_ar4_driver)/config/joint_offsets/$(arg ar_model).yaml"
+    driver_parameters_file="$(find annin_ar4_driver)/config/driver.yaml"
+    tf_prefix="$(arg tf_prefix)"
+  />
 </robot>

File: src/annin_ar4_description/urdf/ar_gazebo.urdf.xacro (robot description, xacro)
@@ -37,5 +37,5 @@
     tf_prefix="$(arg tf_prefix)"
   />
-  <gazebo reference="world" />
+  <!-- <gazebo reference="world" />
   <gazebo>
     <plugin filename="libgz_ros2_control-system" name="gz_ros2_control::GazeboSimROS2ControlPlugin">
@@ -45,4 +45,4 @@
       </ros>
     </plugin>
-  </gazebo>
+  </gazebo> -->
 </robot>
