Commit message: MovIt Works

File: src/annin_ar4_description/urdf/annin_ar4_geometry.urdf (robot description, URDF)
Before this commit: robot annin_ar4, 8 links, 7 joints
Links:
- removed link base_link
Joints:
- removed joint base_link_to_ar4_mk4_motor_17ls13_0404e_200h_c1_1
- joint base_to_link1: child baseplate -> ar4_mk4_j1_turret_housing_1; origin xyz=0.052582 0.147717 -0.05045 rpy=1.5708 0.305123 -0.763446 -> xyz=0.0716069 0.0168825 0.0570797 rpy=-3.14159 5.93e-10 0; parent ar4_mk4_j1_turret_housing_1 -> baseplate
- joint endeffector: origin xyz=0.0189709 -0.00105071 0.0433 rpy=-1.5708 -0.825386 1.51547 -> xyz=-0.00511492 -0.0182986 0.0433 rpy=-1.5708 -0.0993423 -0.272569
- joint endeffector_mount: limit lower=-2.03907 upper=2.14972 effort=10 velocity=10 -> lower=-0.25103 upper=3.93776 effort=10 velocity=10; origin xyz=0.040138 0.0180261 -0.172 rpy=2.71949 1.5708 0 -> xyz=0.0269364 0.0347913 -0.172 rpy=2.22962 1.5708 0
- joint link1_to_link2: child ar4_mk4_j1_turret_housing_1 -> link_2; origin xyz=-0 -0.305 -0.015 rpy=-3.14159 -0 0 -> xyz=0.0202569 -0.0790539 -0.143075 rpy=-1.5708 0.349014 -0.653502; parent link_2 -> ar4_mk4_j1_turret_housing_1
- joint link2_to_link3: child link_2 -> ar4_mk4_motor_17ls13_0404e_200h_c1_1; origin xyz=0.323281 0.133316 0.420505 rpy=1.5708 0.763446 0.305123 -> xyz=0 0.305 0.015 rpy=3.14159 -0 -0; parent ar4_mk4_motor_17ls13_0404e_200h_c1_1 -> link_2
- joint link3_to_end_effector_mount: origin xyz=0.285858 0.0835761 0.420099 rpy=1.56279 -1.78e-10 1.87592 -> xyz=-0.0463871 -0.020311 -0.0362 rpy=-2.72888 -1.5708 0

File: src/annin_ar4_description/urdf/ar.urdf.xacro (robot description, xacro)
@@ -1,9 +1,9 @@
 <?xml version="1.0"?>
 <robot xmlns:xacro="http://wiki.ros.org/xacro" name="$(arg ar_model)">
-  <xacro:arg name="tf_prefix" default="" />
-  <xacro:arg name="include_gripper" default="true"/>
-  <xacro:include filename="$(find annin_ar4_description)/urdf/ar_macro.xacro"/>
+  <!-- <xacro:arg name="tf_prefix" default="" />
+  <xacro:arg name="include_gripper" default="true"/> -->
+  <!-- <xacro:include filename="$(find annin_ar4_description)/urdf/ar_macro.xacro"/> -->
   <xacro:include filename="$(find annin_ar4_description)/urdf/annin_ar4_geometry.urdf"/>
-  <link name="world" />
+  <!-- <link name="world" />
   <xacro:ar_robot
     tf_prefix="$(arg tf_prefix)"
@@ -19,4 +19,4 @@
       parent="$(arg tf_prefix)ee_link"
     />
-  </xacro:if>
+  </xacro:if> -->
 </robot>

Commit message: loads in gazebo, list_controllers broken

File: src/annin_ar4_description/urdf/annin_ar4_geometry.urdf (robot description, URDF)
Before this commit: robot annin_ar4, 7 links, 6 joints
Links:
- link baseplate: mass 0 -> 1

File: src/annin_ar4_description/urdf/ar.urdf.xacro (robot description, xacro)
@@ -1,6 +1,7 @@
 <?xml version="1.0"?>
-<robot xmlns:xacro="http://wiki.ros.org/xacro" name="ar4">
+<robot xmlns:xacro="http://wiki.ros.org/xacro" name="annin_ar4">
   <!-- <xacro:arg name="tf_prefix" default="" />
   <xacro:arg name="include_gripper" default="true"/> -->
+  <!-- <xacro:arg name="tf_prefix" default="" /> -->
   <!-- <xacro:include filename="$(find annin_ar4_description)/urdf/ar_macro.xacro"/> -->
   <xacro:include filename="$(find annin_ar4_description)/urdf/annin_ar4_geometry.urdf"/>
@@ -30,3 +31,14 @@
     />
   </xacro:if> -->
+  <ros2_control name="GazeboSystem" type="system">
+  <hardware>
+    <plugin>gazebo_ros2_control/GazeboSystem</plugin>
+  </hardware>
+  <joint name="head_swivel" />
+</ros2_control>
+<gazebo>
+  <plugin filename="libgazebo_ros2_control.so" name="gazebo_ros2_control">
+    <parameters>$(find urdf_sim_tutorial)/config/09a-minimal.yaml</parameters>
+  </plugin>
+</gazebo>
 </robot>

Commit message: Everything except for the gripper works now

File: src/annin_ar4_description/urdf/annin_ar4_geometry.urdf (robot description, URDF)
Before this commit: robot annin_ar4, 7 links, 6 joints
Links:
- removed link ar4_mk4_14hs11_1004d_egs20_ar4_1
- removed link ar4_mk4_j1_turret_housing_1
- removed link ar4_mk4_motor_17ls13_0404e_200h_c1_1
- removed link link_2
- removed link simplified_part
- removed link simplified_part_2
- added link base_turret_housing, mass 2.54104; visual mesh filename=package://annin_ar4_description/meshes/merged/base_turret_h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
- added link endeffector_part, mass 0.712121; visual mesh filename=package://annin_ar4_description/meshes/merged/endeffector_p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
- added link gripper_motor, mass 0.314103; visual mesh filename=package://annin_ar4_description/meshes/merged/gripper_motor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
- added link gripper_part, mass 0.115892; visual mesh filename=package://annin_ar4_description/meshes/merged/gripper_part_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
- added link link_2_part, mass 0.825114; visual mesh filename=package://annin_ar4_description/meshes/merged/link_2_part_v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
- added link link_6_motor, mass 0.841792; visual mesh filename=package://annin_ar4_description/meshes/merged/link_6_motor_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
- link baseplate: geometry visual mesh filename=package://annin_ar4_description/meshes/merged/baseplate_vis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
Joints:
- joint base_to_link1: child ar4_mk4_j1_turret_housing_1 -> base_turret_housing
- joint endeffector: child simplified_part_2 -> gripper_part; origin xyz=-0.00511492 -0.0182986 0.0433 rpy=-1.5708 -0.0993423 -0.272569 -> xyz=0.019 4.04422e-05 0.0433 rpy=-1.5708 -1.24286 1.57292; parent ar4_mk4_14hs11_1004d_egs20_ar4_1 -> gripper_motor
- joint endeffector_mount: child ar4_mk4_14hs11_1004d_egs20_ar4_1 -> gripper_motor; limit lower=-0.25103 upper=3.93776 effort=10 velocity=10 -> lower=-2.09652 upper=2.09227 effort=10 velocity=10; origin xyz=0.0269364 0.0347913 -0.172 rpy=2.22962 1.5708 0 -> xyz=0.0254835 0.0358691 -0.172 rpy=2.18851 1.5708 0; parent simplified_part -> endeffector_part
- joint link1_to_link2: child link_2 -> link_2_part; origin xyz=0.0202569 -0.0790539 -0.143075 rpy=-1.5708 0.349014 -0.653502 -> xyz=-0.0630431 0.0518211 -0.143075 rpy=-1.5708 1.42706 3.12003; parent ar4_mk4_j1_turret_housing_1 -> base_turret_housing
- joint link2_to_link3: child ar4_mk4_motor_17ls13_0404e_200h_c1_1 -> link_6_motor; origin xyz=0 0.305 0.015 rpy=3.14159 -0 -0 -> xyz=0 0.305 0.015 rpy=3.14159 -0 0; parent link_2 -> link_2_part
- joint link3_to_end_effector_mount: child simplified_part -> endeffector_part; origin xyz=-0.0463871 -0.020311 -0.0362 rpy=-2.72888 -1.5708 0 -> xyz=-0.0284498 -0.0418916 -0.0362 rpy=-2.16738 -1.5708 0; parent ar4_mk4_motor_17ls13_0404e_200h_c1_1 -> link_6_motor
